File: leit-proto-1.brd (EAGLE design)
At the start: 160 x 100 mm, 31 parts, among them J3 FTDI_DEVICE, J4 C-GRID-02-70553, J5 C-GRID-02-70553, J6 C-GRID-02-70553, J7 C-GRID-02-70553, J8 C-GRID-02-70553, J9 M25PTH, Q1 CSD17551Q3A, Q2 CSD17551Q3A, Q3 CSD17551Q3A, Q4 CSD17551Q3A, U1 R-78E5.0-0.5, U2 IR4427S, U3 IR4427S

Commit message: PCB layout complete for barebones proto
Parts:
- moved J8 289.5 mm to (62.7, 94.0)
- moved J7 270.2 mm to (52.8, 94.0)
- moved J6 240.4 mm to (22.6, 94.0)
- moved J4 227.5 mm to (37.8, 94.0)
- moved J5 221.3 mm to (13.0, 94.0)
- moved C1 180.9 mm to (75.2, 82.5), turned to 270 degrees
- moved R3 178.5 mm to (4.83, 87.9)
- moved Q4 176.5 mm to (26.4, 85.1)
- moved R2 174.9 mm to (70.6, 87.6), turned to 180 degrees
- moved R4 173.6 mm to (10.4, 81.5), turned to 270 degrees
- moved Q3 173.6 mm to (16.8, 85.1)
- moved Q2 173.4 mm to (66.5, 85.1)
- moved C4 171.1 mm to (8.38, 82.8), turned to 270 degrees
- moved U2 165.1 mm to (71.6, 82.8)
- moved U3 162.9 mm to (4.57, 83.3)
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Connections:
- removed net N$31: J9.24, MOD1.P$54
- net +5V: now also J9.24, MOD1.P$53, MOD1.P$54
Routing:
- net +12V: track 0.00 -> 186.6 mm, vias 0 -> 3
- net VDD: track 0.00 -> 102.7 mm, vias 0 -> 3
- net +5V: track 0.00 -> 88.4 mm
- net CH3: track 0.00 -> 74.7 mm
- net CH2: track 0.00 -> 68.6 mm
- net AUDIO_L_TAP: track 0.00 -> 56.0 mm
- net AUDIO_R_TAP: track 0.00 -> 45.4 mm
- net GND: track 0.00 -> 39.7 mm, vias 0 -> 12
- net CH0: track 0.00 -> 24.5 mm
- net AUDIO_R: track 0.00 -> 23.1 mm
- net AUDIO_L: track 0.00 -> 20.5 mm
- net CH1_L: track 0.00 -> 19.3 mm
- net N$7: track 0.00 -> 18.8 mm
- net CH1: track 0.00 -> 18.5 mm
- net N$6: track 0.00 -> 16.4 mm
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- added copper zone on layer 1, net CH2_L
- added copper zone on layer 1, net CH3_L
- added copper zone on layer 16, net GND
Other:
- board size 160 x 100 mm -> 77.5 x 100 mm
- board text added: "+"
- board text added: "+12"
- board text added: "0 Red"
- board text added: "1 Grn"
- board text added: "2 Blue"
- board text added: "3 White"
- board text added: "BAT"
- board text added: "BLK"
- board text added: "Flash-o-Matic"
- board text added: "GND"
- board text added: "GRN"
- board text added: "Hank Productions"
